File: PCB/MotorInterface/MotorInterface.kicad_sch (KiCad schematic)
At the start: 9 parts, among them SW1 Switch_SW_Push, U1 74LS193, U2 74LS14, U3 74LS08, U4 74LS193

Commit message: update schema
Parts:
- added C1: TBD, symbol F2018-cache:C
- added D10, D3, D4, D5, D6, D7, D8, D9: LED_small, symbol 00TJR:LED_small
- added D11: G, symbol Drivers-cache:Drivers-rescue_LED-00TJR
- added D12: 1N4001, symbol F2018-cache:D
- added R1, R3: 330, symbol S2020-cache:Device_R_US
- added R4: TBD, symbol S2020-cache:Device_R_US
- added R5: POT, symbol F2018-cache:POT
- added RN1: R_330_DIPx08, Resistor_THT:R_Array_SIP9, symbol 00TJR:R_Pack08_US
- added U5, U6: 74LS76, symbol Counters-cache:74xx_74LS76
- added U7: 74xx_74LS76, symbol S2020-cache:74xx_74LS76
- D2: value Drivers-rescue_LED-00TJR -> R
Connections:
- net A: now also D12.2 (A)
- net GND: now also C1.2, R4.2, U5.1, U5.16 (K), U5.4 (J)
- net VCC: now also D2.2 (A), D11.2 (A)
- net ~{Decrement}: now also U5.3
- net ~{Increment}: now also U5.2
- net at D2.1 (K): now also R1.2
- net ~{D_{0}} renamed D_{0}
- net D_{0}: now also RN1.9
- net ~{D_{1}} renamed D_{1}
- net D_{1}: now also RN1.10
- net ~{D_{2}} renamed D_{2}
- net D_{2}: now also RN1.11
- net ~{D_{3}} renamed D_{3}
- net D_{3}: now also RN1.12
- net ~{D_{4}} renamed D_{4}
- net D_{4}: now also RN1.13
- net ~{D_{5}} renamed D_{5}
- net D_{5}: now also RN1.14
- net ~{D_{6}} renamed D_{6}
- net D_{6}: now also RN1.15
- net ~{D_{7}} renamed D_{7}
- net D_{7}: now also RN1.16
- new net: R1.1, U5.15 (Q)
- new net: D6.1 (K), RN1.5
- new net: D4.1 (K), RN1.7
- new net: R3.1, U5.14
- new net: D11.1 (K), R3.2
- new net: D7.1 (K), RN1.4
- new net: D10.1 (K), RN1.1
- new net: D9.1 (K), RN1.2
- new net: D8.1 (K), RN1.3
- new net: D5.1 (K), RN1.6
- new net: D3.1 (K), RN1.8
- new net: R4.1, R5.2, R5.~
- new net +5V: D10.2 (A), D3.2 (A), D4.2 (A), D5.2 (A), D6.2 (A), D7.2 (A), D8.2 (A), D9.2 (A)
- new net Speed Analog: C1.1, D12.1 (K), R5.1
Other:
- moved on the sheet: C2, D2, R2, SW1

Commit message: update 7476 symbol
Parts:
- removed D1: 00TJR_LED_small, symbol S2020-cache:00TJR_LED_small
- removed U7: 74xx_74LS76, symbol S2020-cache:74xx_74LS76
- added C3: TBD, symbol F2018-cache:C
- added R6: TBD, symbol S2020-cache:Device_R_US
- U2: renamed from U6; symbol Counters-cache:74xx_74LS76 -> 00TJR:74xx_74LS76
Connections:
- net GND: now also U2.13 (GND), C3.2
- net Speed Analog: now also C3.1, R6.2; no longer C1.1, D12.1 (K)
- net VCC: now also U2.5 (VCC)
- new net: C1.1, D12.1 (K), R6.1
Other:
- moved on the sheet: C1, C2, D12, R2, R4, R5, SW1
