File: PCB/Anderson Projects/Pico_H-bridge_complete/power.kicad_sch (KiCad schematic)
At the start: 19 parts, among them U2 OPA4197, U3 LM7810, U4 LM79L05

Commit message: Made new Anderson PCB project and reverted Tim R's folder
Parts:
- removed U4: LM79L05, Package_TO_SOT_THT:TO-92_Inline, symbol Regulator_Linear:LM78L05_TO92
- added U7: LM78L05_SO8, Package_SO:SOIC-8_3.9x4.9mm_P1.27mm, symbol Regulator_Linear:LM78L05_SO8
- C10: renamed from C11; footprint TJR:C_Radial_D5.00mm_H12.5mm_P2.00mm -> Capacitor_Tantalum_SMD:CP_EIA-3216-10_Kemet-I; symbol TJR:C_Polarized_US -> Device:C_Polarized_US
- C11: renamed from C14; footprint TJR:C_Rect_L7.3mm_W2.5_H6.5mm_P5.0mm -> Capacitor_SMD:C_0805_2012Metric
- C12: renamed from C6; footprint TJR:C_Radial_D5.00mm_H12.5mm_P2.00mm -> Capacitor_Tantalum_SMD:CP_EIA-3216-10_Kemet-I; symbol TJR:C_Polarized_US -> Device:C_Polarized_US
- C13: renamed from C9; footprint TJR:C_Rect_L7.3mm_W2.5_H6.5mm_P5.0mm -> Capacitor_SMD:C_0805_2012Metric
- C14: renamed from C12; footprint TJR:C_Radial_D5.00mm_H12.5mm_P2.00mm -> Capacitor_Tantalum_SMD:CP_EIA-3216-10_Kemet-I; symbol TJR:C_Polarized_US -> Device:C_Polarized_US
- C15, C17, C19: footprint TJR:C_Rect_L7.3mm_W2.5_H6.5mm_P5.0mm -> Capacitor_SMD:C_0805_2012Metric
- C16, C18, C4: footprint TJR:C_Radial_D5.00mm_H12.5mm_P2.00mm -> Capacitor_Tantalum_SMD:CP_EIA-3216-10_Kemet-I; symbol TJR:C_Polarized_US -> Device:C_Polarized_US
- C5: renamed from C7; footprint TJR:C_Rect_L7.3mm_W2.5_H6.5mm_P5.0mm -> Capacitor_SMD:C_0805_2012Metric
- C6: renamed from C10; footprint TJR:C_Radial_D5.00mm_H12.5mm_P2.00mm -> Capacitor_Tantalum_SMD:CP_EIA-3216-10_Kemet-I; symbol TJR:C_Polarized_US -> Device:C_Polarized_US
- C7: renamed from C13; footprint TJR:C_Rect_L7.3mm_W2.5_H6.5mm_P5.0mm -> Capacitor_SMD:C_0805_2012Metric
- C8: renamed from C5; footprint TJR:C_Radial_D5.00mm_H12.5mm_P2.00mm -> Capacitor_Tantalum_SMD:CP_EIA-3216-10_Kemet-I; symbol TJR:C_Polarized_US -> Device:C_Polarized_US
- C9: renamed from C8; footprint TJR:C_Rect_L7.3mm_W2.5_H6.5mm_P5.0mm -> Capacitor_SMD:C_0805_2012Metric
- U5: renamed from U2; footprint TJR:D14_TEX -> CustomBPA:SO-14_5.4_P1.27
- U6: renamed from U3; footprint Package_TO_SOT_THT:TO-220-3_Vertical -> Package_SO:SOIC-8_3.9x4.9mm_P1.27mm; symbol Regulator_Linear:LM7810_TO220 -> Regulator_Linear:L78L10_SO8
Connections:
- net +10V: now also U6.1 (OUT), U7.8 (IN); no longer U6.3 (VO)
- net +5V: now also U7.1 (OUT)
- net GND: now also U6.3 (GND), U6.6 (GND), U6.7 (GND), U7.2 (GND), U7.3 (GND), U7.6 (GND), U7.7 (GND)
- net +12V renamed +Vsup
- net +Vsup: now also U6.8 (IN); no longer U6.1 (VI)

Commit message: Changed Dig inputs  to zener buffers, removed all opto-couples, rebuilt h-bridge logic.
Parts:
- removed C19: 0.1uF, Capacitor_SMD:C_0805_2012Metric, symbol Device:C
- added C21: 1uF, Capacitor_SMD:C_1206_3216Metric, symbol Device:C
- C10, C12, C14, C16, C18, C4, C6, C8: footprint Capacitor_Tantalum_SMD:CP_EIA-3216-10_Kemet-I -> Capacitor_SMD:C_1210_3225Metric
- C11, C13, C15, C17, C5, C7, C9: footprint Capacitor_SMD:C_0805_2012Metric -> Capacitor_SMD:C_0603_1608Metric
Connections:
- net +3.3V: now also C21.1
- net GND: now also C21.2
Other:
- note added: "1uF and 0.1uF placed as close to Pico ADC_VREF"
