File: PCB/MotorInterfaceDiscrete/MotorInterface.kicad_sch (KiCad schematic)
At the start: 30 parts, among them SW1 Switch_SW_Push, U1 74LS193, U2 74LS76, U3 74LS14, U4 74LS08, U5 74LS193, U6 74LS193

Commit message: update schema notes
Other:
- note added: "Encoder Position Counter - 12 bit Resolution"
- note added: "Encoder Pulse to Analog Voltage with Adjust"
- note added: "Encoder State Detectors & Pulse Generators"
- note added: "Latch To Indicate Direction"
- note added: "Position/Direction Indicatiors and Home Reset Manual/Power Up"
Changed lines of the file:
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@@
+    (stroke (width 0) (type default))
+  )
+  (polyline (pts (xy 199.39 168.91) (xy 265.43 168.91))
     (stroke (width 0) (type default))
   )
@@
     (stroke (width 0) (type default))
   )
+  (polyline (pts (xy 200.66 60.96) (xy 246.38 60.96))
+    (stroke (width 0) (type default))
+  )
   (wire (pts (xy 140.97 162.56) (xy 138.43 162.56))
     (stroke (width 0) (type default))
@@
     (stroke (width 0) (type default))
   )
+  (polyline (pts (xy 59.69 200.66) (xy 106.68 200.66))
+    (stroke (width 0) (type default))
+  )
   (wire (pts (xy 237.49 100.33) (xy 234.95 100.33))
     (stroke (width 0) (type default))
@@
   )
   (wire (pts (xy 71.12 53.34) (xy 74.93 53.34))
+    (stroke (width 0) (type default))
+  )
+  (polyline (pts (xy 100.33 67.31) (xy 146.05 67.31))
     (stroke (width 0) (type default))
   )
@@
     (stroke (width 0) (type default))
   )
+  (polyline (pts (xy 31.75 113.03) (xy 60.96 113.03))
+    (stroke (width 0) (type default))
+  )
   (wire (pts (xy 194.31 100.33) (xy 194.31 110.49))
     (stroke (width 0) (type default))
@@
     (stroke (width 0) (type default))
   )
+  (text "Encoder Position Counter - 12 bit Resolution" (at 60.96 199.39 0)
+    (effects (font (size 1.27 1.27) (thickness 0.254) bold) (justify left bottom))
+  )
+  (text "Encoder State Detectors & Pulse Generators" (at 101.6 66.04 0)
+    (effects (font (size 1.27 1.27) (thickness 0.254) bold) (justify left bottom))
+  )
+  (text "Encoder Pulse to Analog Voltage with Adjust" (at 201.93 59.69 0)
+    (effects (font (size 1.27 1.27) (thickness 0.254) bold) (justify left bottom))
+  )
+  (text "Latch To Indicate Direction" (at 33.02 111.76 0)
+    (effects (font (size 1.27 1.27) (thickness 0.254) bold) (justify left bottom))
+  )
+  (text "Position/Direction Indicatiors and Home Reset Manual/Power Up"
+    (at 200.66 167.64 0)
+    (effects (font (size 1.27 1.27) (thickness 0.254) bold) (justify left bottom))
+  )
   (global_label "D_{0}" (shape output) (at 63.5 149.86 0) (fields_autoplaced)

Commit message: update symbols, add decouple
Parts:
- U1, U5, U6: value 74LS193 -> 74HC193; symbol S2020-cache:74LS193 -> 00TJR:74HC193
Connections:
- net GND: no longer U1.8 (GND), U5.8 (GND), U6.8 (GND)
- net VCC: no longer U1.16 (VCC), U5.16 (VCC), U6.16 (VCC)

Commit message: add tested analog speed circuit
Parts:
- added C14: 1uF, symbol F2018-cache:C
- added Q1: BS170, Package_TO_SOT_THT:TO-92_Inline, symbol 00TJR:BS170_copy
- added Q2: 2N3906, Package_TO_SOT_THT:TO-92_Inline, symbol 00TJR:2N3906
- added R1: 1k, symbol S2020-cache:Device_R_US
- added R2: 100, symbol S2020-cache:Device_R_US
- added R4: 33k, symbol S2020-cache:Device_R_US
- C1: value TBD -> 0.1uF
- C2: value TBD -> 0.33uF
- R3: value TBD -> 10k
- R5: renamed from R1; value TBD -> 100
- R6: renamed from R2; value POT -> 22k
Connections:
- net GND: now also R6.1, C14.2, Q1.3 (S), R1.2, R2.2; no longer C1.2, R3.2
- net Speed Analog: now also R6.2, R6.~, C14.1; no longer C2.1, R6.1
- net at C1.1, D4.1 (K): now also R1.1; no longer R5.1
- new net: C1.2, Q1.2 (G), R2.1
- new net: Q1.1 (D), R3.2, R4.1
- new net: Q2.~ (E), R4.2
- new net: C2.1, Q2.~ (E), R5.1
- new net V+: Q2.~ (E), R3.1
Other:
- note added: "0-100k"
- moved on the sheet: C1, C2, D4, R5, R6
