File: PCB/MotorInterfaceShootout/MotorInterfaceShootout.kicad_sch (KiCad schematic)
At the start: 31 parts, among them J1 Screw_Terminal_01x10, J2 Motor Connector, U1 Pico, U2 OPA4197

Commit message: ready for footprints
Parts:
- removed D1, D2, D3, D4, D5, D8, D9: 3V, symbol TJR:ZENER
- added R15, R16, R21, R22: 820, symbol TJR:R
- added R30, R31: 5.1k, symbol TJR:R
- R2: value 1k -> 2.55k; digikey https://www.digikey.com/en/products/detail/stackpole-electronics-inc/RMCF0805FT1K00/1760090 -> https://www.digikey.com/en/products/detail/stackpole-electronics-inc/RMCF0805FG2K55/1712818
- U1: digikey https://www.digikey.com/en/products/detail/texas-instrument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 -> (none)
Connections:
- net A: now also R30.2
- net B: now also R31.2
- net GND: now also R15.2, R16.2, R21.2, R22.2, R30.1, R31.1
- net PIN_HOME_CMD: now also R16.1
- net PIN_HOME_LIMIT: now also R15.1
- net S0_PLC: now also R21.1
- net S1_PLC: now also R22.1
Other:
- moved on the sheet: R2, R3

Commit message: most footprints, added and measured/confirmed
Parts:
- D6, D7: footprint (none) -> LED_SMD:LED_0805_2012Metric_Pad1.15x1.40mm_HandSolder
- R1, R10, R11, R12, R13, R15, R16, R2, R21, R22, R24, R3, R30, R31, R4, R5, R6, R7, R8, R9: footprint (none) -> R_SMD:R_0805_2012Metric
Changed lines of the file:
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@@
 			)
 		)
-		(property "Footprint" ""
+		(property "Footprint" "R_SMD:R_0805_2012Metric"
 			(at 66.04 142.748 90)
 			(effects
@@
 			)
 		)
-		(property "Footprint" ""
+		(property "Footprint" "R_SMD:R_0805_2012Metric"
 			(at 124.46 45.72 0)
 			(effects
@@
 			)
 		)
-		(property "Footprint" ""
+		(property "Footprint" "R_SMD:R_0805_2012Metric"
 			(at 70.612 144.78 90)
 			(effects
@@
 			)
 		)
-		(property "Footprint" ""
+		(property "Footprint" "R_SMD:R_0805_2012Metric"
 			(at 70.612 182.88 90)
 			(effects
@@
 			)
 		)
-		(property "Footprint" ""
+		(property "Footprint" "R_SMD:R_0805_2012Metric"
 			(at 70.612 170.18 90)
 			(effects
@@
 			)
 		)
-		(property "Footprint" ""
+		(property "Footprint" "R_SMD:R_0805_2012Metric"
 			(at 66.04 130.048 90)
 			(effects
@@
 			)
 		)
-		(property "Footprint" ""
+		(property "Footprint" "R_SMD:R_0805_2012Metric"
 			(at 250.19 140.208 90)
 			(effects
@@
 			)
 		)
-		(property "Footprint" ""
+		(property "Footprint" "R_SMD:R_0805_2012Metric"
 			(at 258.318 154.94 90)
 			(effects
@@
 			)
 		)
-		(property "Footprint" ""
+		(property "Footprint" "R_SMD:R_0805_2012Metric"
 			(at 66.04 155.448 90)
 			(effects
@@
 			)
 		)
-		(property "Footprint" ""
+		(property "Footprint" "R_SMD:R_0805_2012Metric"
 			(at 223.52 60.198 90)
 			(effects
@@
 			)
 		)
-		(property "Footprint" ""
+		(property "Footprint" "R_SMD:R_0805_2012Metric"
 			(at 250.19 152.908 90)
 			(effects
@@
 			)
 		)
-		(property "Footprint" ""
+		(property "Footprint" "R_SMD:R_0805_2012Metric"
 			(at 224.79 93.218 90)
 			(effects
@@
 			)
 		)
-		(property "Footprint" ""
+		(property "Footprint" "R_SMD:R_0805_2012Metric"
 			(at 153.162 91.44 90)
 			(effects
@@
 			)
 		)
-		(property "Footprint" ""
+		(property "Footprint" "R_SMD:R_0805_2012Metric"
 			(at 258.318 142.24 90)
 			(effects
@@
 			)
 		)
-		(property "Footprint" ""
+		(property "Footprint" "R_SMD:R_0805_2012Metric"
 			(at 66.04 168.148 90)
 			(effects
@@
 			)
 		)
-		(property "Footprint" ""
+		(property "Footprint" "R_SMD:R_0805_2012Metric"
 			(at 146.812 91.44 90)
 			(effects
@@
 			)
 		)
-		(property "Footprint" ""
+		(property "Footprint" "R_SMD:R_0805_2012Metric"
 			(at 223.52 28.448 90)
 			(effects
@@
 			)
 		)
-		(property "Footprint" ""
+		(property "Footprint" "R_SMD:R_0805_2012Metric"
 			(at 66.04 180.848 90)
 			(effects
@@
 			)
 		)
-		(property "Footprint" ""
+		(property "Footprint" "LED_SMD:LED_0805_2012Metric_Pad1.15x1.40mm_HandSolder"
 			(at 154.94 100.33 90)
 			(effects
@@
 			)
 		)
-		(property "Footprint" ""
+		(property "Footprint" "R_SMD:R_0805_2012Metric"
 			(at 70.612 157.48 90)
 			(effects
@@
 			)
 		)
-		(property "Footprint" ""
+		(property "Footprint" "LED_SMD:LED_0805_2012Metric_Pad1.15x1.40mm_HandSolder"
 			(at 148.59 100.33 90)
 			(effects
@@
 			)
 		)
-		(property "Footprint" ""
+		(property "Footprint" "R_SMD:R_0805_2012Metric"
 			(at 70.612 132.08 90)
 			(effects

Commit message: all footprints
Parts:
- removed J1: Screw_Terminal_01x10, symbol connector:Screw_Terminal_01x10
- added J3: Screw_Terminal_01x02, Screw_Term:TerminalBlock_WAGO_236-102_1x02_P5.00mm_45Degree, symbol connector:Screw_Terminal_01x02
- added J4: Screw_Terminal_01x08, Screw_Term:TerminalBlock_WAGO_236-108_1x08_P5.00mm_45Degree, symbol connector:Screw_Terminal_01x08
- JP1: footprint (none) -> Header-IDC:PinHeader_1x02_P2.54mm_Vertical
Connections:
- net GND: now also J3.1 (Pin_1)
- net PIN_PWM_POS: now also J4.7 (Pin_7)
- net PIN_PWM_POSX10: now also J4.6 (Pin_6)
- net PIN_PWM_SPD: now also J4.8 (Pin_8)
- net at R1.1: now also J4.4 (Pin_4)
- net at R24.1: now also J4.5 (Pin_5)
- net at R5.1: now also J4.1 (Pin_1)
- net at R4.1: now also J4.2 (Pin_2)
- net at R3.1: now also J4.3 (Pin_3)
- new net +VSYS: J3.2 (Pin_2)

Commit message: fix trim pot footprint
Parts:
- R7: footprint R_SMD:R_0805_2012Metric -> TJR:SOT_10KLFTR_BIT
Changed lines of the file:
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@@
 			)
 		)
-		(property "Footprint" "R_SMD:R_0805_2012Metric"
+		(property "Footprint" "TJR:SOT_10KLFTR_BIT"
 			(at 124.46 45.72 0)
 			(effects

Commit message: continue four layer layout
Parts:
- J3: renamed from J2; footprint Connector_JST:JST_XH_B6B-XH-A_1x06_P2.50mm_Vertical -> jst:JST_XH_B6B-XH-A_1x06_P2.50mm_Vertical
- R17: renamed from R6; value 5.1k -> 2.55k
- R18: renamed from R13; value 5.1k -> 2.55k
- renumbered D6 to D1, D7 to D2, J3 to J1, J4 to J2, R24 to R1, R22 to R10, R7 to R11, R8 to R12, R9 to R13, R10 to R14, R11 to R15, R12 to R16, R30 to R19, R1 to R2, R31 to R20, R15 to R6, R16 to R7, R2 to R8, R21 to R9
Connections:
- net E+ is gone; now on net +5V: J3.3 (Pin_3)
- net E- is gone; now on net GND: J3.4 (Pin_4)
- net Analog Position: now also J2.7 (Pin_7)
- net Analog Position x10: now also J2.6 (Pin_6)
- net Analog Speed: now also J2.8 (Pin_8)
- net PIN_PWM_POS: no longer J2.7 (Pin_7)
- net PIN_PWM_POSX10: no longer J2.6 (Pin_6)
- net PIN_PWM_SPD: no longer J2.8 (Pin_8)
- net PIN_FWD: no longer names the net of R12.1, U1.21 (GPIO16)
- net PIN_REV: no longer names the net of R13.1, U1.22 (GPIO17)
- net S0_PLC renamed S0
- net S1_PLC renamed S1
Other:
- moved on the sheet: D1, D2, R12, R13
