File: PCB/MotorInterfaceShootout/h-bridge.kicad_sch (KiCad schematic)
At the start: 26 parts, among them Q2 2N7002, Q3 2N7002, Q5 G160P03KI, Q6 G20N03K, Q7 G160P03KI, Q8 G20N03K, U5 74LS14, U6 74LS08

Commit message: all footprints
Parts:
- removed Q7: G160P03KI, symbol Drivers-rescue:PEMOSFET-00TJR
- removed Q8: G20N03K, symbol Drivers-rescue:NEMOSFET-00TJR
- added Q1: G160P03KI, TO_SOT_SMD:TO-252-2, symbol Drivers-rescue:PEMOSFET-00TJR
- added Q4: G20N03K, TO_SOT_SMD:TO-252-2, symbol Drivers-rescue:NEMOSFET-00TJR
- JP2, JP3, JP4: footprint (none) -> Header-IDC:PinHeader_1x02_P2.54mm_Vertical
- Q5, Q6: footprint (none) -> TO_SOT_SMD:TO-252-2
- U5, U6: footprint (none) -> TJR:SOIC-14_3.9x8.7mm_P1.27mm-D14-L
Connections:
- net Forward0: now also Q2.1 (G); no longer Q2.2 (G)
- net Forward1: now also Q4.1 (G)
- net GND: now also Q2.2 (S), Q3.2 (S), Q4.3 (S); no longer Q2.3 (S), Q3.3 (S)
- net M+: now also Q5.2 (D), Q6.2 (D); no longer Q5.3 (D), Q6.1 (D)
- net M-: now also Q1.2 (D), Q4.2 (D)
- net Reverse0: now also Q3.1 (G); no longer Q3.2 (G)
- net Reverse1: now also Q6.1 (G); no longer Q6.2 (G)
- net at R19.1, R23.2: now also Q5.1 (G); no longer Q5.2 (G)
- net at R28.1, R29.2: now also Q1.1 (G)
- net at R23.1: now also Q2.3 (D); no longer Q2.1 (D)
- net at R29.1: now also Q3.3 (D); no longer Q3.1 (D)
- net VSYS renamed +VSYS
- net +VSYS: now also Q5.3 (S), Q1.3 (S); no longer Q5.1 (S)

Commit message: continue four layer layout
Parts:
- R29: renamed from R23; value 5.1k -> 2.55k
- R31: renamed from R29; value 5.1k -> 2.55k
- renumbered C10 to C12, D14 to D4, D15 to D5, D18 to D6, D16 to D7, JP4 to JP3, JP3 to JP4, Q2 to Q1, Q5 to Q2, Q6 to Q3, Q3 to Q4, Q1 to Q5, Q4 to Q6, R17 to R23, R14 to R24, R19 to R28, R28 to R30
Changed lines of the file:
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@@
 		(on_board yes)
 		(dnp no)
-		(property "Reference" "Q6"
+		(property "Reference" "Q3"
 			(at 204.216 151.384 0)
 			(effects
@@
 			(project "MotorInterfaceShootout"
 				(path "/00c452e7-2941-4e66-a1a1-d4af87d7e63e/0acf8530-81b2-4261-9d60-47f6831c6925"
-					(reference "Q6")
+					(reference "Q3")
 					(unit 1)
 				)
@@
 		(on_board yes)
 		(dnp no)
-		(property "Reference" "Q5"
+		(property "Reference" "Q2"
 			(at 204.47 91.694 0)
 			(effects
@@
 			(project "MotorInterfaceShootout"
 				(path "/00c452e7-2941-4e66-a1a1-d4af87d7e63e/0acf8530-81b2-4261-9d60-47f6831c6925"
-					(reference "Q5")
+					(reference "Q2")
 					(unit 1)
 				)
@@
 		(on_board yes)
 		(dnp no)
-		(property "Reference" "D18"
+		(property "Reference" "D6"
 			(at 84.582 134.366 0)
 			(effects
@@
 			(project "MotorInterfaceShootout"
 				(path "/00c452e7-2941-4e66-a1a1-d4af87d7e63e/0acf8530-81b2-4261-9d60-47f6831c6925"
-					(reference "D18")
+					(reference "D6")
 					(unit 1)
 				)
@@
 		(on_board yes)
 		(dnp no)
-		(property "Reference" "Q4"
+		(property "Reference" "Q6"
 			(at 263.906 151.384 0)
 			(effects
@@
 			(project "MotorInterfaceShootout"
 				(path "/00c452e7-2941-4e66-a1a1-d4af87d7e63e/0acf8530-81b2-4261-9d60-47f6831c6925"
-					(reference "Q4")
+					(reference "Q6")
 					(unit 1)
 				)
@@
 		(on_board yes)
 		(dnp no)
-		(property "Reference" "Q2"
+		(property "Reference" "Q1"
 			(at 193.04 109.728 0)
 			(effects
@@
 			(project "MotorInterfaceShootout"
 				(path "/00c452e7-2941-4e66-a1a1-d4af87d7e63e/0acf8530-81b2-4261-9d60-47f6831c6925"
-					(reference "Q2")
+					(reference "Q1")
 					(unit 1)
 				)
@@
 		(on_board yes)
 		(dnp no)
-		(property "Reference" "#PWR041"
+		(property "Reference" "#PWR040"
 			(at 81.28 130.81 0)
 			(effects
@@
 			(project "MotorInterfaceShootout"
 				(path "/00c452e7-2941-4e66-a1a1-d4af87d7e63e/0acf8530-81b2-4261-9d60-47f6831c6925"
-					(reference "#PWR041")
+					(reference "#PWR040")
 					(unit 1)
 				)
@@
 		(on_board yes)
 		(dnp no)
-		(property "Reference" "#PWR040"
+		(property "Reference" "#PWR039"
 			(at 81.28 115.57 0)
 			(effects
@@
 			(project "MotorInterfaceShootout"
 				(path "/00c452e7-2941-4e66-a1a1-d4af87d7e63e/0acf8530-81b2-4261-9d60-47f6831c6925"
-					(reference "#PWR040")
+					(reference "#PWR039")
 					(unit 1)
 				)
@@
 		(on_board yes)
 		(dnp no)
-		(property "Reference" "R28"
+		(property "Reference" "R30"
 			(at 251.206 89.662 0)
 			(effects
@@
 			(project "MotorInterfaceShootout"
 				(path "/00c452e7-2941-4e66-a1a1-d4af87d7e63e/0acf8530-81b2-4261-9d60-47f6831c6925"
-					(reference "R28")
+					(reference "R30")
 					(unit 1)
 				)
@@
 		(on_board yes)
 		(dnp no)
-		(property "Reference" "D14"
+		(property "Reference" "D4"
 			(at 83.82 104.14 90)
 			(effects
@@
 			(project "MotorInterfaceShootout"
 				(path "/00c452e7-2941-4e66-a1a1-d4af87d7e63e/0acf8530-81b2-4261-9d60-47f6831c6925"
-					(reference "D14")
+					(reference "D4")
 					(unit 1)
 				)
@@
 		(on_board yes)
 		(dnp no)
-		(property "Reference" "#PWR036"
+		(property "Reference" "#PWR046"
 			(at 252.73 124.46 0)
 			(effects
@@
 			(project "MotorInterfaceShootout"
 				(path "/00c452e7-2941-4e66-a1a1-d4af87d7e63e/0acf8530-81b2-4261-9d60-47f6831c6925"
-					(reference "#PWR036")
+					(reference "#PWR046")
 					(unit 1)
 				)
@@
 		(on_board yes)
 		(dnp no)
-		(property "Reference" "#PWR035"
+		(property "Reference" "#PWR038"
 			(at 71.12 43.18 0)
 			(effects
@@
 			(project "MotorInterfaceShootout"
 				(path "/00c452e7-2941-4e66-a1a1-d4af87d7e63e/0acf8530-81b2-4261-9d60-47f6831c6925"
-					(reference "#PWR035")
+					(reference "#PWR038")
 					(unit 1)
 				)
@@
 		(on_board yes)
 		(dnp no)
-		(property "Reference" "Q1"
+		(property "Reference" "Q5"
 			(at 264.16 91.694 0)
 			(effects
@@
 			(project "MotorInterfaceShootout"
 				(path "/00c452e7-2941-4e66-a1a1-d4af87d7e63e/0acf8530-81b2-4261-9d60-47f6831c6925"
-					(reference "Q1")
+					(reference "Q5")
 					(unit 1)
 				)
@@
 		(on_board yes)
 		(dnp no)
-		(property "Reference" "R23"
+		(property "Reference" "R29"
 			(at 190.5 100.076 0)
 			(effects
@@
 			)
 		)
-		(property "Value" "5.1k"
+		(property "Value" "2.55k"
 			(at 191.008 101.854 0)
 			(effects
@@
 			(project "MotorInterfaceShootout"
 				(path "/00c452e7-2941-4e66-a1a1-d4af87d7e63e/0acf8530-81b2-4261-9d60-47f6831c6925"
-					(reference "R23")
+					(reference "R29")
 					(unit 1)
 				)
@@
 		(on_board yes)
 		(dnp no)
-		(property "Reference" "JP4"
+		(property "Reference" "JP3"
 			(at 223.52 131.064 0)
 			(effects
@@
 			(project "MotorInterfaceShootout"
 				(path "/00c452e7-2941-4e66-a1a1-d4af87d7e63e/0acf8530-81b2-4261-9d60-47f6831c6925"
-					(reference "JP4")
+					(reference "JP3")
 					(unit 1)
 				)
@@
 		(on_board yes)
 		(dnp no)
-		(property "Reference" "D15"
+		(property "Reference" "D5"
 			(at 83.82 119.38 90)
 			(effects
@@
 			(project "MotorInterfaceShootout"
 				(path "/00c452e7-2941-4e66-a1a1-d4af87d7e63e/0acf8530-81b2-4261-9d60-47f6831c6925"
-					(reference "D15")
+					(reference "D5")
 					(unit 1)
 				)
@@
 		(on_board yes)
 		(dnp no)
-		(property "Reference" "R29"
+		(property "Reference" "R31"
 			(at 251.206 99.822 0)
 			(effects
@@
 			)
 		)
-		(property "Value" "5.1k"
+		(property "Value" "2.55k"
 			(at 251.714 101.6 0)
 			(effects
@@
 			(project "MotorInterfaceShootout"
 				(path "/00c452e7-2941-4e66-a1a1-d4af87d7e63e/0acf8530-81b2-4261-9d60-47f6831c6925"
-					(reference "R29")
+					(reference "R31")
 					(unit 1)
 				)
@@
 		(on_board yes)
 		(dnp no)
-		(property "Reference" "#PWR043"
+		(property "Reference" "#PWR042"
 			(at 81.28 161.29 0)
 			(effects
@@
 			(project "MotorInterfaceShootout"
 				(path "/00c452e7-2941-4e66-a1a1-d4af87d7e63e/0acf8530-81b2-4261-9d60-47f6831c6925"
-					(reference "#PWR043")
+					(reference "#PWR042")
 					(unit 1)
 				)
@@
 		(on_board yes)
 		(dnp no)
-		(property "Reference" "C10"
+		(property "Reference" "C12"
 			(at 236.982 141.732 90)
 			(effects
@@
 			(project ""
 				(path "/00c452e7-2941-4e66-a1a1-d4af87d7e63e/0acf8530-81b2-4261-9d60-47f6831c6925"
-					(reference "C10")
+					(reference "C12")
 					(unit 1)
 				)
@@
 		(on_board yes)
 		(dnp no)
-		(property "Reference" "D16"
+		(property "Reference" "D7"
 			(at 84.582 149.606 0)
 			(effects
@@
 			(project "MotorInterfaceShootout"
 				(path "/00c452e7-2941-4e66-a1a1-d4af87d7e63e/0acf8530-81b2-4261-9d60-47f6831c6925"
-					(reference "D16")
+					(reference "D7")
 					(unit 1)
 				)
@@
 		(on_board yes)
 		(dnp no)
-		(property "Reference" "#PWR034"
+		(property "Reference" "#PWR043"
 			(at 191.77 124.46 0)
 			(effects
@@
 			(project "MotorInterfaceShootout"
 				(path "/00c452e7-2941-4e66-a1a1-d4af87d7e63e/0acf8530-81b2-4261-9d60-47f6831c6925"
-					(reference "#PWR034")
+					(reference "#PWR043")
 					(unit 1)
 				)
@@
 		(on_board yes)
 		(dnp no)
-		(property "Reference" "#PWR039"
+		(property "Reference" "#PWR047"
 			(at 262.89 166.37 0)
 			(effects
@@
 			(project "MotorInterfaceShootout"
 				(path "/00c452e7-2941-4e66-a1a1-d4af87d7e63e/0acf8530-81b2-4261-9d60-47f6831c6925"
-					(reference "#PWR039")
+					(reference "#PWR047")
 					(unit 1)
 				)
@@
 		(on_board yes)
 		(dnp no)
-		(property "Reference" "R14"
+		(property "Reference" "R24"
 			(at 76.708 99.314 90)
 			(effects
@@
 			(project "MotorInterfaceShootout"
 				(path "/00c452e7-2941-4e66-a1a1-d4af87d7e63e/0acf8530-81b2-4261-9d60-47f6831c6925"
-					(reference "R14")
+					(reference "R24")
 					(unit 1)
 				)
@@
 		(on_board yes)
 		(dnp no)
-		(property "Reference" "#PWR038"
+		(property "Reference" "#PWR044"
 			(at 203.2 166.37 0)
 			(effects
@@
 			(project "MotorInterfaceShootout"
 				(path "/00c452e7-2941-4e66-a1a1-d4af87d7e63e/0acf8530-81b2-4261-9d60-47f6831c6925"
-					(reference "#PWR038")
+					(reference "#PWR044")
 					(unit 1)
 				)
@@
 		(on_board yes)
 		(dnp no)
-		(property "Reference" "Q3"
+		(property "Reference" "Q4"
 			(at 254 109.728 0)
 			(effects
@@
 			(project "MotorInterfaceShootout"
 				(path "/00c452e7-2941-4e66-a1a1-d4af87d7e63e/0acf8530-81b2-4261-9d60-47f6831c6925"
-					(reference "Q3")
+					(reference "Q4")
 					(unit 1)
 				)
@@
 		(on_board yes)
 		(dnp no)
-		(property "Reference" "JP3"
+		(property "Reference" "JP4"
 			(at 223.52 141.224 0)
 			(effects
@@
 			(project "MotorInterfaceShootout"
 				(path "/00c452e7-2941-4e66-a1a1-d4af87d7e63e/0acf8530-81b2-4261-9d60-47f6831c6925"
-					(reference "JP3")
+					(reference "JP4")
 					(unit 1)
 				)
@@
 		(on_board yes)
 		(dnp no)
-		(property "Reference" "R17"
+		(property "Reference" "R23"
 			(at 69.85 41.148 0)
 			(effects
@@
 			(project "MotorInterfaceShootout"
 				(path "/00c452e7-2941-4e66-a1a1-d4af87d7e63e/0acf8530-81b2-4261-9d60-47f6831c6925"
-					(reference "R17")
+					(reference "R23")
 					(unit 1)
 				)
@@
 		(on_board yes)
 		(dnp no)
-		(property "Reference" "#PWR042"
+		(property "Reference" "#PWR041"
 			(at 81.28 146.05 0)
 			(effects
@@
 			(project "MotorInterfaceShootout"
 				(path "/00c452e7-2941-4e66-a1a1-d4af87d7e63e/0acf8530-81b2-4261-9d60-47f6831c6925"
-					(reference "#PWR042")
+					(reference "#PWR041")
 					(unit 1)
 				)
@@
 		(on_board yes)
 		(dnp no)
-		(property "Reference" "R19"
+		(property "Reference" "R28"
 			(at 190.5 89.408 0)
 			(effects
@@
 			(project "MotorInterfaceShootout"
 				(path "/00c452e7-2941-4e66-a1a1-d4af87d7e63e/0acf8530-81b2-4261-9d60-47f6831c6925"
-					(reference "R19")
+					(reference "R28")
 					(unit 1)
 				)
