File: PCB/MotorInterfaceShootout/power.kicad_sch (KiCad schematic)
At the start: 19 parts, among them U2 OPA4197, U3 LM7810, U4 LM79L05

Commit message: fix power
Parts:
- removed C10, C11, C12, C16, C18: 100uF, TJR:C_Radial_D5.00mm_H12.5mm_P2.00mm, symbol TJR:C_Polarized_US
- removed C13, C14, C15, C17, C19, C7, C8, C9: 0.1uF, TJR:C_Rect_L7.3mm_W2.5_H6.5mm_P5.0mm, symbol Device:C
Connections:
- net +12V renamed VSYS
Other:
- note removed: "Decoupling Networks Note: Place nearest component power pins"
- moved on the sheet: C4

Commit message: working on h-bridge logic
Parts:
- added R1, R12: 10k, TJR:R_Axial_DIN0207_L6.3mm_D2.5mm_P7.62mm_Horizontal, symbol TJR:R
Connections:
- net +5V: now also R1.1
- net GND: now also R12.2
- new net COMP_THRES: R1.2, R12.1
Other:
- note added: "Op-Amp Comparator Threshold Voltage Note: must be less digital IO pin voltage out"

Commit message: ready for cleanup and layout
Parts:
- added U5: 74LS14, symbol S2020-cache:74xx_74LS14
- added U9: 74LS08, symbol TFlipFlop-cache:74xx_74LS08
Changed lines of the file:
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@@
+	)
+	(symbol
+		(lib_id "TFlipFlop-cache:74xx_74LS08")
+		(at 110.49 82.55 0)
+		(mirror x)
+		(unit 5)
+		(exclude_from_sim no)
+		(in_bom yes)
+		(on_board yes)
+		(dnp no)
+		(property "Reference" "U9"
+			(at 109.22 87.63 0)
+			(effects
+				(font
+					(size 1.27 1.27)
+				)
+			)
+		)
+		(property "Value" "74LS08"
+			(at 110.49 88.9 0)
+			(effects
+				(font
+					(size 1.27 1.27)
+				)
+				(hide yes)
+			)
+		)
+		(property "Footprint" ""
+			(at 110.49 82.55 0)
+			(effects
+				(font
+					(size 1.27 1.27)
+				)
+				(hide yes)
+			)
+		)
+		(property "Datasheet" ""
+			(at 110.49 82.55 0)
+			(effects
+				(font
+					(size 1.27 1.27)
+				)
+				(hide yes)
+			)
+		)
+		(property "Description" ""
+			(at 110.49 82.55 0)
+			(effects
+				(font
+					(size 1.27 1.27)
+				)
+				(hide yes)
+			)
+		)
+		(property "Cost (ea.)" ""
+			(at 110.49 82.55 0)
+			(effects
+				(font
+					(size 1.27 1.27)
+				)
+				(hide yes)
+			)
+		)
+		(property "Vender Part Number" ""
+			(at 110.49 82.55 0)
+			(effects
+				(font
+					(size 1.27 1.27)
+				)
+				(hide yes)
+			)
+		)
+		(pin "13"
+		)
+		(pin "1"
+		)
+		(pin "10"
+		)
+		(pin "9"
+		)
+		(pin "3"
+		)
+		(pin "7"
+		)
+		(pin "11"
+		)
+		(pin "14"
+		)
+		(pin "12"
+		)
+		(pin "5"
+		)
+		(pin "8"
+		)
+		(pin "2"
+		)
+		(pin "6"
+		)
+		(pin "4"
+		)
+		(instances
+			(project "MotorInterfaceShootout"
+				(path "/00c452e7-2941-4e66-a1a1-d4af87d7e63e/4eca7562-021b-4add-9e83-06681ce2d496"
+					(reference "U9")
+					(unit 5)
+				)
+			)
+		)
 	)
 	(symbol
@@
 					(reference "#PWR022")
 					(unit 1)
+				)
+			)
+		)
+	)
+	(symbol
+		(lib_id "S2020-cache:74xx_74LS14")
+		(at 92.71 80.01 0)
+		(mirror x)
+		(unit 7)
+		(exclude_from_sim no)
+		(in_bom yes)
+		(on_board yes)
+		(dnp no)
+		(property "Reference" "U5"
+			(at 94.488 77.216 0)
+			(effects
+				(font
+					(size 1.27 1.27)
+				)
+			)
+		)
+		(property "Value" "74LS14"
+			(at 92.71 86.36 0)
+			(effects
+				(font
+					(size 1.27 1.27)
+				)
+				(hide yes)
+			)
+		)
+		(property "Footprint" ""
+			(at 92.71 80.01 0)
+			(effects
+				(font
+					(size 1.27 1.27)
+				)
+				(hide yes)
+			)
+		)
+		(property "Datasheet" ""
+			(at 92.71 80.01 0)
+			(effects
+				(font
+					(size 1.27 1.27)
+				)
+				(hide yes)
+			)
+		)
+		(property "Description" ""
+			(at 92.71 80.01 0)
+			(effects
+				(font
+					(size 1.27 1.27)
+				)
+				(hide yes)
+			)
+		)
+		(property "Cost (ea.)" ""
+			(at 92.71 80.01 0)
+			(effects
+				(font
+					(size 1.27 1.27)
+				)
+				(hide yes)
+			)
+		)
+		(property "Vender Part Number" ""
+			(at 92.71 80.01 0)
+			(effects
+				(font
+					(size 1.27 1.27)
+				)
+				(hide yes)
+			)
+		)
+		(pin "11"
+		)
+		(pin "13"
+		)
+		(pin "12"
+		)
+		(pin "7"
+		)
+		(pin "14"
+		)
+		(pin "9"
+		)
+		(pin "5"
+		)
+		(pin "10"
+		)
+		(pin "8"
+		)
+		(pin "3"
+		)
+		(pin "1"
+		)
+		(pin "2"
+		)
+		(pin "6"
+		)
+		(pin "4"
+		)
+		(instances
+			(project "MotorInterfaceShootout"
+				(path "/00c452e7-2941-4e66-a1a1-d4af87d7e63e/4eca7562-021b-4add-9e83-06681ce2d496"
+					(reference "U5")
+					(unit 7)
 				)
 			)
@@
 		)
 		(property "Value" "LM79L05"
-			(at 92.964 29.718 0)
-			(effects
-				(font
+			(at 88.392 16.256 0)
+			(effects
+				(font

Commit message: working on part source
Parts:
- removed U3: LM7810, Package_TO_SOT_THT:TO-220-3_Vertical, symbol Regulator_Linear:LM7810_TO220
- added C7, C8, C9: 0.1uF, symbol device:C
- added U3: L78L10ACUTR, symbol Regulator_Linear:LM78L05_TO92
- C4, C5, C6: footprint TJR:C_Radial_D5.00mm_H12.5mm_P2.00mm -> (none); digikey https://www.digikey.com/en/products/detail/rubycon/16ZLH100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 -> https://www.digikey.com/en/products/detail/nichicon/UWT1V10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
- R15: renamed from R1; footprint TJR:R_Axial_DIN0207_L6.3mm_D2.5mm_P7.62mm_Horizontal -> (none); digikey https://www.digikey.com/en/products/detail/stackpole-electronics-inc/CFM12JT47R0/1741962 -> https://www.digikey.com/en/products/detail/stackpole-electronics-inc/RMCF0805FT10K0/1760676
- R16: renamed from R12; footprint TJR:R_Axial_DIN0207_L6.3mm_D2.5mm_P7.62mm_Horizontal -> (none); digikey https://www.digikey.com/en/products/detail/stackpole-electronics-inc/CFM12JT47R0/1741962 -> https://www.digikey.com/en/products/detail/stackpole-electronics-inc/RMCF0805FT10K0/1760676
- U4: value LM79L05 -> L78L05ABUTR; footprint Package_TO_SOT_THT:TO-92_Inline -> (none); digikey https://www.digikey.com/en/products/detail/texas-instrument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 -> https://www.digikey.com/en/products/detail/stmicroelectroni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
- U5: digikey (none) -> https://www.digikey.com/en/products/detail/texas-instrument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
- U6: renamed from U9; digikey (none) -> https://www.digikey.com/en/products/detail/texas-instrument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
Connections:
- net +10V: now also U4.3 (VI), C7.1, U3.1 (VO); no longer U4.1 (VO)
- net +5V: now also U4.1 (VO), U5.14 (VCC), U6.14 (VCC), C8.1, C9.1; no longer U4.3 (VI)
- net GND: now also U5.7 (GND), U6.7 (GND), C7.2, C8.2, C9.2, U3.2 (GND)
- net VSYS: now also U3.3 (VI)
Other:
- moved on the sheet: U5G, U6E

Commit message: ready for footprints
Parts:
- removed C5, C6: 100uF, symbol TJR:C_Polarized_US
- removed R15, R16: 10k, symbol TJR:R
- added C12, C5, C6: 0.1uF, symbol device:C
- added R18, R20: 5.1k, symbol TJR:R
Connections:
- net +10V: now also C12.1, C5.1
- net +5V: now also C6.1, R18.2
- net COMP_THRES: now also R18.1, R20.2
- net GND: now also C12.2, C5.2, C6.2, R20.1
Other:
- moved on the sheet: C4, U3, U4

Commit message: most footprints, added and measured/confirmed
Parts:
- C12, C5, C6, C7, C8, C9: footprint (none) -> C_SMD:C_0805_2012Metric
- C4: footprint (none) -> C_SMD:CP_Elec_6.3x7.7
- R18, R20: footprint (none) -> R_SMD:R_0805_2012Metric
- U3, U4: footprint (none) -> TO_SOT_SMD:SOT-89-3
Changed lines of the file:
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@@
 			)
 		)
-		(property "Footprint" ""
+		(property "Footprint" "C_SMD:CP_Elec_6.3x7.7"
 			(at 44.1452 41.91 0)
 			(effects
@@
 			)
 		)
-		(property "Footprint" ""
+		(property "Footprint" "C_SMD:C_0805_2012Metric"
 			(at 243.5352 85.09 0)
 			(effects
@@
 			)
 		)
-		(property "Footprint" ""
+		(property "Footprint" "R_SMD:R_0805_2012Metric"
 			(at 222.758 26.67 90)
 			(effects
@@
 			)
 		)
-		(property "Footprint" ""
+		(property "Footprint" "R_SMD:R_0805_2012Metric"
 			(at 222.758 36.83 90)
 			(effects
@@
 			)
 		)
-		(property "Footprint" ""
+		(property "Footprint" "C_SMD:C_0805_2012Metric"
 			(at 69.5452 41.91 0)
 			(effects
@@
 			)
 		)
-		(property "Footprint" ""
+		(property "Footprint" "TO_SOT_SMD:SOT-89-3"
 			(at 55.88 27.305 0)
 			(effects
@@
 			)
 		)
-		(property "Footprint" ""
+		(property "Footprint" "C_SMD:C_0805_2012Metric"
 			(at 129.2352 39.37 0)
 			(effects
@@
 			)
 		)
-		(property "Footprint" ""
+		(property "Footprint" "C_SMD:C_0805_2012Metric"
 			(at 219.4052 85.09 0)
 			(effects
@@
 			)
 		)
-		(property "Footprint" ""
+		(property "Footprint" "TO_SOT_SMD:SOT-89-3"
 			(at 96.52 27.305 0)
 			(effects
@@
 			)
 		)
-		(property "Footprint" ""
+		(property "Footprint" "C_SMD:C_0805_2012Metric"
 			(at 82.2452 41.91 0)
 			(effects
@@
 			)
 		)
-		(property "Footprint" ""
+		(property "Footprint" "C_SMD:C_0805_2012Metric"
 			(at 111.4552 41.91 0)
 			(effects

Commit message: all footprints
Parts:
- added D1: MSS1P4, D_SMD:D_MicroSMP_AK, symbol device:D_Filled
- U5, U6: footprint (none) -> TJR:SOIC-14_3.9x8.7mm_P1.27mm-D14-L
Connections:
- net VSYS: no longer names the net of C4.1, U3.3 (VI)
- net VSYS: now also D1.1 (K)
- new net +VSYS: D1.2 (A)
Changed lines of the file:
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@@
-	)
-	(junction
-		(at 43.18 44.45)
-		(diameter 0)
-		(color 0 0 0 0)
 	)
 	(junction
@@
 	(wire
 		(pts
-			(xy 36.83 44.45) (xy 43.18 44.45)
-		)
-		(stroke
-			(width 0)
-			(type default)
-		)
-	)
-	(wire
-		(pts
 			(xy 139.7 26.67) (xy 139.7 27.94)
 		)
@@
 	(wire
 		(pts
+			(xy 29.21 33.02) (xy 25.4 33.02)
+		)
+		(stroke
+			(width 0)
+			(type default)
+		)
+	)
+	(wire
+		(pts
 			(xy 218.44 67.31) (xy 208.28 67.31)
 		)
@@
 		(pts
 			(xy 63.5 33.02) (xy 68.58 33.02)
+		)
+		(stroke
+			(width 0)
+			(type default)
+		)
+	)
+	(wire
+		(pts
+			(xy 25.4 33.02) (xy 25.4 26.67)
 		)
 		(stroke
@@
 				)
 				(justify left)
-				(hide yes)
-			)
-		)
-	)
-	(global_label "GND"
-		(shape input)
-		(at 36.83 44.45 180)
-		(fields_autoplaced yes)
-		(effects
-			(font
-				(size 1.27 1.27)
-			)
-			(justify right)
-		)
-		(property "Intersheetrefs" "${INTERSHEET_REFS}"
-			(at 29.9743 44.45 0)
-			(effects
-				(font
-					(size 1.27 1.27)
-				)
-				(justify right)
-				(hide yes)
-			)
-		)
-	)
-	(global_label "VSYS"
-		(shape input)
-		(at 36.83 33.02 180)
-		(fields_autoplaced yes)
-		(effects
-			(font
-				(size 1.27 1.27)
-			)
-			(justify right)
-		)
-		(property "Intersheetrefs" "${INTERSHEET_REFS}"
-			(at 29.2486 33.02 0)
-			(effects
-				(font
-					(size 1.27 1.27)
-				)
-				(justify right)
 				(hide yes)
 			)
@@
 			)
 		)
-		(property "Footprint" ""
+		(property "Footprint" "TJR:SOIC-14_3.9x8.7mm_P1.27mm-D14-L"
 			(at 232.41 81.28 0)
 			(effects
@@
 				(path "/00c452e7-2941-4e66-a1a1-d4af87d7e63e/4eca7562-021b-4add-9e83-06681ce2d496"
 					(reference "C9")
+					(unit 1)
+				)
+			)
+		)
+	)
+	(symbol
+		(lib_id "device:D_Filled")
+		(at 33.02 33.02 0)
+		(mirror y)
+		(unit 1)
+		(exclude_from_sim no)
+		(in_bom yes)
+		(on_board yes)
+		(dnp no)
+		(property "Reference" "D1"
+			(at 33.02 27.94 0)
+			(effects
+				(font
+					(size 1.27 1.27)
+				)
+			)
+		)
+		(property "Value" "MSS1P4"
+			(at 33.02 30.48 0)
+			(effects
+				(font
+					(size 1.27 1.27)
+				)
+			)
+		)
+		(property "Footprint" "D_SMD:D_MicroSMP_AK"
+			(at 33.02 33.02 0)
+			(effects
+				(font
+					(size 1.27 1.27)
+				)
+				(hide yes)
+			)
+		)
+		(property "Datasheet" "https://www.vishay.com/docs/89019/mss1p4.pdf"
+			(at 33.02 33.02 0)
+			(effects
+				(font
+					(size 1.27 1.27)
+				)
+				(hide yes)
+			)
+		)
+		(property "Description" "DIODE SCHOTTKY 40V 1A DO219AD"
+			(at 33.02 33.02 0)
+			(effects
+				(font
+					(size 1.27 1.27)
+				)
+				(hide yes)
+			)
+		)
+		(property "Sim.Device" "D"
+			(at 33.02 33.02 0)
+			(effects
+				(font
+					(size 1.27 1.27)
+				)
+				(hide yes)
+			)
+		)
+		(property "Sim.Pins" "1=K 2=A"
+			(at 33.02 33.02 0)
+			(effects
+				(font
+					(size 1.27 1.27)
+				)
+				(hide yes)
+			)
+		)
+		(property "digikey" "https://www.digikey.com/en/products/detail/vishay-general-semiconductor-diodes-division/MSS1P4-M3-89A/2071753"
+			(at 33.02 33.02 0)
+			(effects
+				(font
+					(size 1.27 1.27)
+				)
+				(hide yes)
+			)
+		)
+		(pin "1"
+		)
+		(pin "2"
+		)
+		(instances
+			(project ""
+				(path "/00c452e7-2941-4e66-a1a1-d4af87d7e63e/4eca7562-021b-4add-9e83-06681ce2d496"
+					(reference "D1")
 					(unit 1)
 				)
@@
 			)
 		)
-		(property "Footprint" ""
+		(property "Footprint" "TJR:SOIC-14_3.9x8.7mm_P1.27mm-D14-L"
 			(at 208.28 81.28 0)
 			(effects
@@
 					(unit 1)
 				)
+			)
+		)
+	)
+	(symbol
+		(lib_id "power:+3.3V")
+		(at 25.4 26.67 0)
+		(unit 1)
+		(exclude_from_sim no)
+		(in_bom yes)
+		(on_board yes)
+		(dnp no)
+		(property "Reference" "#PWR044"
+			(at 25.4 30.48 0)
+			(effects
+				(font
+					(size 1.27 1.27)
+				)
+				(hide yes)
+			)
+		)
+		(property "Value" "+VSYS"
+			(at 25.4 22.86 0)
+			(effects
+				(font
+					(size 1.27 1.27)
+				)
+			)
+		)
+		(property "Footprint" ""
+			(at 25.4 26.67 0)
+			(effects
+				(font
+					(size 1.27 1.27)
+				)
+				(hide yes)
+			)
+		)
+		(property "Datasheet" ""
+			(at 25.4 26.67 0)
+			(effects
+				(font
+					(size 1.27 1.27)
+				)
+				(hide yes)
+			)
+		)
+		(property "Description" "+5V to +30V"
+			(at 25.4 26.67 0)
+			(effects
+				(font
+					(size 1.27 1.27)
+				)
+				(hide yes)
+			)
+		)
+		(pin "1"
+		)
+		(instances
+			(project "MotorInterfaceShootout"
+				(path "/00c452e7-2941-4e66-a1a1-d4af87d7e63e/4eca7562-021b-4add-9e83-06681ce2d496"
+					(reference "#PWR044")
+					(unit 1)
+				)

Commit message: continue four layer layout
Parts:
- removed R20: 5.1k, R_SMD:R_0805_2012Metric, symbol TJR:R
- added R22: 820, R_SMD:R_0805_2012Metric, symbol TJR:R
- renumbered C9 to C10, C12 to C6, C6 to C7, C7 to C8, C8 to C9, D1 to D3, R18 to R21
Connections:
- net +10V: now also R21.2
- net +5V: no longer R21.2
- net COMP_THRES: now also R22.1
- net GND: now also R22.2
Other:
- note added: "Op-Amp Comparator Threshold Voltage Note: must be less digital IO pin voltage out high (Voh)"
- note removed: "Op-Amp Comparator Threshold Voltage Note: must be less digital IO pin voltage out"
